Commit message: changes to topics

File: src/my_robot/urdf/my_robot.xacro (robot description, xacro)
@@ -1,210 +1,231 @@
-<?xml version='1.0'?>
-<robot name="my_robot"
-  xmlns:xacro="http://www.ros.org/wiki/xacro">
-  <xacro:include filename="$(find my_robot)/urdf/my_robot.gazebo" />
-  <link name="robot_footprint"></link>
-  <joint name="robot_footprint_joint" type="fixed">
-    <origin xyz="0 0 0" rpy="0 0 0" />
-    <parent link="robot_footprint"/>
-    <child link="chassis" />
+<?xml version="1.0"?>
+<robot name="my_robot" xmlns:xacro="http://www.ros.org/wiki/xacro">
+	<include filename="$(find my_robot)/urdf/my_robot.gazebo" />
+	<link name="robot_footprint">
+	</link>
+	<joint name="robot_footprint_joint" type="fixed">
+		<origin xyz="0 0 0" rpy="0 0 0" />
+		<parent link="robot_footprint" />
+		<child link="chassis" />
+	</joint>
+	<joint name="camera_joint" type="fixed">
+		<origin xyz="0.15 0.0 0.2" rpy="0 0.25 0" />
+		<axis xyz="0 1 0" rpy="0 0 0" />
+		<parent link="chassis" />
+		<child link="camera" />
+	</joint>
+	<joint name="hokuyo_joint" type="fixed">
+		<origin xyz="0.11 0.0 0.075" rpy="0 0 0" />
+		<axis xyz="0 1 0" rpy="0 0 0" />
+		<parent link="chassis" />
+		<child link="hokuyo" />
+	</joint>
+	<joint type="continuous" name="left_wheel_hinge">
+		<origin xyz="0.0 0.18 0" rpy="0 0 0" />
+		<child link="left_wheel" />
+		<parent link="chassis" />
+		<axis xyz="0 1 0" rpy="0 0 0" />
+		<limit effort="10000" velocity="1000" />
+		<dynamics damping="1.0" friction="1.0" />
+	</joint>
+	<joint type="continuous" name="right_wheel_hinge">
+		<origin xyz="0.0 -0.18 0" rpy="0 0 0" />
+		<child link="right_wheel" />
+		<parent link="chassis" />
+		<axis xyz="0 1 0" rpy="0 0 0" />
+		<limit effort="10000" velocity="1000" />
+		<dynamics damping="1.0" friction="1.0" />
+	</joint>
+  <joint name="camera_optical_joint" type="fixed">
+    <origin xyz="0 0 0" rpy="-1.5707 0 -1.5707"/>
+    <parent link="camera"/>
+    <child link="camera_link_optical"/>
   </joint>
-  <joint name="camera_joint" type="fixed">
-    <origin xyz="0.15 0.0 0.2" rpy="0 0.25 0" />
-    <axis xyz="0 1 0" rpy="0 0 0"/>
-    <parent link="chassis"/>
-    <child link="camera" />
-  </joint>
-  <joint name="hokuyo_joint" type="fixed">
-    <origin xyz="0.11 0.0 0.075" rpy="0 0 0" />
-    <axis xyz="0 1 0" rpy="0 0 0"/>
-    <parent link="chassis"/>
-    <child link="hokuyo" />
-  </joint>
-  <joint type="continuous" name="left_wheel_hinge">
-    <origin xyz="0.0 0.18 0" rpy="0 0 0"/>
-    <child link="left_wheel"/>
-    <parent link="chassis"/>
-    <axis xyz="0 1 0" rpy="0 0 0"/>
-    <limit effort="10000" velocity="1000"/>
-    <dynamics damping="1.0" friction="1.0"/>
-  </joint>
-  <joint type="continuous" name="right_wheel_hinge">
-    <origin xyz="0.0 -0.18 0" rpy="0 0 0"/>
-    <child link="right_wheel"/>
-    <parent link="chassis"/>
-    <axis xyz="0 1 0" rpy="0 0 0"/>
-    <limit effort="10000" velocity="1000"/>
-    <dynamics damping="1.0" friction="1.0"/>
-  </joint>
-  <link name='chassis'>
-    <pose>0 0 0.1 0 0 0</pose>
-    <inertial>
-      <mass value="15.0"/>
-      <origin xyz="0.0 0 0" rpy=" 0 0 0"/>
-      <inertia ixx="0.1" ixy="0" ixz="0" iyy="0.1" iyz="0" izz="0.1" />
-    </inertial>
-    <collision name='bottom_chassis_collision'>
-      <origin xyz="0 0 0" rpy=" 0 0 0"/>
-      <geometry>
-        <cylinder radius="0.16" length="0.08"/>
-      </geometry>
-    </collision>
-    <visual name='bottom_chassis_visual'>
-      <origin xyz="0 0 0" rpy=" 0 0 0"/>
-      <geometry>
-        <cylinder radius="0.15" length="0.08"/>
-      </geometry>
-    </visual>
-    <collision name='top_chassis_collision'>
-      <origin xyz="0 0 0.2" rpy=" 0 0 0"/>
-      <geometry>
-        <cylinder radius="0.16" length="0.08"/>
-      </geometry>
-    </collision>
-    <visual name='top_chassis_visual'>
-      <origin xyz="0 0 0.2" rpy=" 0 0 0"/>
-      <geometry>
-        <cylinder radius="0.15" length="0.08"/>
-      </geometry>
-    </visual>
-    <collision name='front_caster_collision'>
-      <origin xyz="0.10 0 -0.03" rpy=" 0 0 0"/>
-      <geometry>
-        <sphere radius="0.06"/>
-      </geometry>
-    </collision>
-    <visual name='front_caster_visual'>
-      <origin xyz="0.10 0 -0.03" rpy=" 0 0 0"/>
-      <geometry>
-        <sphere radius="0.06"/>
-      </geometry>
-    </visual>
-    <collision name='back_caster_collision'>
-      <origin xyz="-0.1 0 -0.03" rpy=" 0 0 0"/>
-      <geometry>
-        <sphere radius="0.06"/>
-      </geometry>
-    </collision>
-    <visual name='back_caster_visual'>
-      <origin xyz="-0.1 0 -0.03" rpy=" 0 0 0"/>
-      <geometry>
-        <sphere radius="0.06"/>
-      </geometry>
-    </visual>
-    <collision name='back_right_pin_collision'>
-      <origin xyz="-0.09 -0.09 0.09" rpy=" 0 0 0"/>
-      <geometry>
-        <cylinder radius="0.01" length="0.3"/>
-      </geometry>
-    </collision>
-    <visual name='back_right_pin_visual'>
-      <origin xyz="-0.09 -0.09 0.09" rpy=" 0 0 0"/>
-      <geometry>
-        <cylinder radius="0.01" length="0.3"/>
-      </geometry>
-    </visual>
-    <collision name='back_left_pin_collision'>
-      <origin xyz="-0.09 0.09 0.09" rpy=" 0 0 0"/>
-      <geometry>
-        <cylinder radius="0.01" length="0.3"/>
-      </geometry>
-    </collision>
-    <visual name='back_left_pin_visual'>
-      <origin xyz="-0.09 0.09 0.09" rpy=" 0 0 0"/>
-      <geometry>
-        <cylinder radius="0.01" length="0.3"/>
-      </geometry>
-    </visual>
+  <link name="camera_link_optical">
   </link>
-  <gazebo reference="chassis">
-    <material>Gazebo/Blue</material>
-  </gazebo>
-  <link name='left_wheel'>
-    <pose>0 0 0.1 0 0 0</pose>
-    <inertial>
-      <mass value="5.0"/>
-      <origin xyz="0.0 0 0" rpy=" 0 1.5707 1.5707"/>
-      <inertia ixx="0.1" ixy="0" ixz="0" iyy="0.1" iyz="0" izz="0.1" />
-    </inertial>
-    <collision name='collision'>
-      <origin xyz="0 0 0" rpy=" 0 1.5707 1.5707"/>
-      <geometry>
-        <cylinder radius="0.092" length="0.04"/>
-      </geometry>
-    </collision>
-    <visual name='left_wheel_visual'>
-      <origin xyz="0 0 0" rpy=" 0 1.5707 1.5707"/>
-      <geometry>
-        <cylinder radius="0.092" length="0.04"/>
-      </geometry>
-    </visual>
-  </link>
-  <gazebo reference="left_wheel">
-    <material>Gazebo/Blue</material>
-  </gazebo>
-  <link name='right_wheel'>
-    <pose>0 0 0.1 0 0 0</pose>
-    <inertial>
-      <mass value="5.0"/>
-      <origin xyz="0.0 0 0" rpy=" 0 1.5707 1.5707"/>
-      <inertia ixx="0.1" ixy="0" ixz="0" iyy="0.1" iyz="0" izz="0.1" />
-    </inertial>
-    <collision name='collision'>
-      <origin xyz="0 0 0" rpy=" 0 1.5707 1.5707"/>
-      <geometry>
-        <cylinder radius="0.092" length="0.04"/>
-      </geometry>
-    </collision>
-    <visual name='right_wheel_visual'>
-      <origin xyz="0 0 0" rpy=" 0 1.5707 1.5707"/>
-      <geometry>
-        <cylinder radius="0.092" length="0.04"/>
-      </geometry>
-    </visual>
-  </link>
-  <gazebo reference="right_wheel">
-    <material>Gazebo/Blue</material>
-  </gazebo>
-  <link name='camera'>
-    <box_inertia m="0.1" x="0.05" y="0.05" z="0.05" />
-    <inertial>
-      <mass value="0.1"/>
-      <origin xyz="0 0 0" rpy=" 0 0 0"/>
-      <inertia ixx="1e-6" ixy="0" ixz="0" iyy="1e-6" iyz="0" izz="1e-6" />
-    </inertial>
-    <collision name='collision'>
-      <origin xyz="0 0 0" rpy=" 0 0 0"/>
-      <geometry>
-        <box size="0.05 0.05 0.05"/>
-      </geometry>
-    </collision>
-    <visual name='camera_visual'>
-      <origin xyz="0 0 0" rpy=" 0 0 0"/>
-      <geometry>
-        <box size="0.05 0.05 0.05"/>
-      </geometry>
-    </visual>
-  </link>
-  <gazebo reference="camera">
-    <material>Gazebo/Green</material>
-  </gazebo>
-  <link name='hokuyo'>
-    <inertial>
-      <mass value="1e-5"/>
-      <origin xyz="0 0 0" rpy=" 0 0 0"/>
-      <inertia ixx="1e-6" ixy="0" ixz="0" iyy="1e-6" iyz="0" izz="1e-6"/>
-    </inertial>
-    <collision name='collision'>
-      <origin xyz="0 0 0" rpy=" 0 0 0"/>
-      <geometry>
-        <box size="0.1 0.1 0.1"/>
-      </geometry>
-    </collision>
-    <visual name='hokuyo_visual'>
-      <origin xyz="0 0 0" rpy=" 0 0 0"/>
-      <geometry>
-        <mesh filename="package://my_robot/meshes/hokuyo.dae"/>
-      </geometry>
-    </visual>
-  </link>
+	<link name="chassis">
+		<pose>
+			0 0 0.1 0 0 0
+		</pose>
+		<inertial>
+			<mass value="15.0" />
+			<origin xyz="0.0 0 0" rpy=" 0 0 0" />
+			<inertia ixx="0.1" ixy="0" ixz="0" iyy="0.1" iyz="0" izz="0.1" />
+		</inertial>
+		<collision name="bottom_chassis_collision">
+			<origin xyz="0 0 0" rpy=" 0 0 0" />
+			<geometry>
+				<cylinder radius="0.16" length="0.08" />
+			</geometry>
+		</collision>
+		<visual name="bottom_chassis_visual">
+			<origin xyz="0 0 0" rpy=" 0 0 0" />
+			<geometry>
+				<cylinder radius="0.15" length="0.08" />
+			</geometry>
+		</visual>
+		<collision name="top_chassis_collision">
+			<origin xyz="0 0 0.2" rpy=" 0 0 0" />
+			<geometry>
+				<cylinder radius="0.16" length="0.08" />
+			</geometry>
+		</collision>
+		<visual name="top_chassis_visual">
+			<origin xyz="0 0 0.2" rpy=" 0 0 0" />
+			<geometry>
+				<cylinder radius="0.15" length="0.08" />
+			</geometry>
+		</visual>
+		<collision name="front_caster_collision">
+			<origin xyz="0.10 0 -0.03" rpy=" 0 0 0" />
+			<geometry>
+				<sphere radius="0.06" />
+			</geometry>
+		</collision>
+		<visual name="front_caster_visual">
+			<origin xyz="0.10 0 -0.03" rpy=" 0 0 0" />
+			<geometry>
+				<sphere radius="0.06" />
+			</geometry>
+		</visual>
+		<collision name="back_caster_collision">
+			<origin xyz="-0.1 0 -0.03" rpy=" 0 0 0" />
+			<geometry>
+				<sphere radius="0.06" />
+			</geometry>
+		</collision>
+		<visual name="back_caster_visual">
+			<origin xyz="-0.1 0 -0.03" rpy=" 0 0 0" />
+			<geometry>
+				<sphere radius="0.06" />
+			</geometry>
+		</visual>
+		<collision name="back_right_pin_collision">
+			<origin xyz="-0.09 -0.09 0.09" rpy=" 0 0 0" />
+			<geometry>
+				<cylinder radius="0.01" length="0.3" />
+			</geometry>
+		</collision>
+		<visual name="back_right_pin_visual">
+			<origin xyz="-0.09 -0.09 0.09" rpy=" 0 0 0" />
+			<geometry>
+				<cylinder radius="0.01" length="0.3" />
+			</geometry>
+		</visual>
+		<collision name="back_left_pin_collision">
+			<origin xyz="-0.09 0.09 0.09" rpy=" 0 0 0" />
+			<geometry>
+				<cylinder radius="0.01" length="0.3" />
+			</geometry>
+		</collision>
+		<visual name="back_left_pin_visual">
+			<origin xyz="-0.09 0.09 0.09" rpy=" 0 0 0" />
+			<geometry>
+				<cylinder radius="0.01" length="0.3" />
+			</geometry>
+		</visual>
+	</link>
+	<gazebo reference="chassis">
+		<material>
+			Gazebo/Blue
+		</material>
+	</gazebo>
+	<link name="left_wheel">
+		<pose>
+			0 0 0.1 0 0 0
+		</pose>
+		<inertial>
+			<mass value="5.0" />
+			<origin xyz="0.0 0 0" rpy=" 0 1.5707 1.5707" />
+			<inertia ixx="0.1" ixy="0" ixz="0" iyy="0.1" iyz="0" izz="0.1" />
+		</inertial>
+		<collision name="collision">
+			<origin xyz="0 0 0" rpy=" 0 1.5707 1.5707" />
+			<geometry>
+				<cylinder radius="0.092" length="0.04" />
+			</geometry>
+		</collision>
+		<visual name="left_wheel_visual">
+			<origin xyz="0 0 0" rpy=" 0 1.5707 1.5707" />
+			<geometry>
+				<cylinder radius="0.092" length="0.04" />
+			</geometry>
+		</visual>
+	</link>
+	<gazebo reference="left_wheel">
+		<material>
+			Gazebo/Blue
+		</material>
+	</gazebo>
+	<link name="right_wheel">
+		<pose>
+			0 0 0.1 0 0 0
+		</pose>
+		<inertial>
+			<mass value="5.0" />
+			<origin xyz="0.0 0 0" rpy=" 0 1.5707 1.5707" />
+			<inertia ixx="0.1" ixy="0" ixz="0" iyy="0.1" iyz="0" izz="0.1" />
+		</inertial>
+		<collision name="collision">
+			<origin xyz="0 0 0" rpy=" 0 1.5707 1.5707" />
+			<geometry>
+				<cylinder radius="0.092" length="0.04" />
+			</geometry>
+		</collision>
+		<visual name="right_wheel_visual">
+			<origin xyz="0 0 0" rpy=" 0 1.5707 1.5707" />
+			<geometry>
+				<cylinder radius="0.092" length="0.04" />
+			</geometry>
+		</visual>
+	</link>
+	<gazebo reference="right_wheel">
+		<material>
+			Gazebo/Blue
+		</material>
+	</gazebo>
+	<link name="camera">
+		<box_inertia m="0.1" x="0.05" y="0.05" z="0.05" />
+		<inertial>
+			<mass value="0.1" />
+			<origin xyz="0 0 0" rpy=" 0 0 0" />
+			<inertia ixx="1e-6" ixy="0" ixz="0" iyy="1e-6" iyz="0" izz="1e-6" />
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